File: Board/Rev1/pico2-ice.kicad_pcb (KiCad board)
At the start: 4 copper layers, 27.9 x 63.5 mm, 123 parts, among them J1 USB_C_Receptacle_USB2.0, J2 Conn_02x20_Odd_Even, J3 Conn_02x20_Odd_Even, J5 BM03B-SRSS-TB, J6 SFV22R-2STE1HLF, SW1 CS1213AGF260, SW2 CS1213AGF260, U1 NCP115AMX120TCG, U2 W25Q32JVSSIQ, U3 RP2350_80QFN, U4 TL431DBZ, U5 APS6404L-3SQN-SN, U6 ICE40UP5K-SG48ITR, U8 W25Q32JVSSIQ, U9 NCP115AMX330TCG, Y1 ABM8-272-T3

Commit message: pico2-ice gerber
Parts:
- moved C6 2.07 mm to (73.1, 103.4), turned to 0 degrees
- moved R23 1.01 mm to (77.4, 98.0), turned to -90 degrees
- moved R13 0.74 mm to (78.5, 96.6), turned to 90 degrees
Routing:
- net /SCL_GPIO3: track 47.1 -> 59.7 mm, vias 3 -> 4
- net /GPIO10: track 0.00 -> 11.7 mm, vias 0 -> 2
- net /GPIO11: track 0.00 -> 11.3 mm, vias 0 -> 2
- net /Lane0_P: track 0.00 -> 9.46 mm
- net /Lane0_N: track 0.59 -> 9.50 mm
- net /Clock_P: track 0.59 -> 9.46 mm
- net /Lane1_N: track 0.59 -> 9.38 mm
- net /Lane1_P: track 0.66 -> 9.38 mm
- net /Clock_N: track 1.23 -> 9.51 mm
- net +3V3: track 81.7 -> 90.0 mm
- net /Lane2_N: track 2.65 -> 10.1 mm
- net /Lane2_P: track 2.78 -> 10.1 mm
- net GND: track 49.3 -> 54.8 mm, vias 60 -> 62
- net /LED_R: track 44.1 -> 39.8 mm, vias 3 -> 2
- net /ICE_25: track 51.2 -> 55.4 mm
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Other:
- board text added: "0"
- board text added: "0 mm"
- board text added: "0.01 mm"
- board text added: "0.0152 mm"
- board text added: "0.02"
- board text added: "0.035 mm"
- board text added: "0.0994 mm"
- board text added: "0.14097"
- board text added: "0.1524"
- board text added: "0.1524 mm / 0.1270 mm"
- board text added: "0.2540 mm"
- board text added: "1"
- board text added: "1.265 mm"
- board text added: "1.5842 mm"
- board text added: "100 OHM DIFF"
- board text added: "27.9410 mm x 63.5005 mm"
- board text added: "4.05"
- board text added: "50 OHM SE"
- board text added: "B.Cu"
- board text added: "B.Mask"
- board text added: "B.Paste"
- board text added: "B.Silkscreen"
- board text added: "BOARD CHARACTERISTICS"
- board text added: "BOTTOM"
- board text added: "Board Thickness:"
- board text added: "Board overall dimensions:"
- board text added: "Bottom Silk Screen"
- board text added: "Bottom Solder Mask"
- board text added: "Bottom Solder Paste"
- board text added: "Castellated pads:"
- board text added: "Color"
- board text added: "Copper Finish:"
- board text added: "Copper Layer Count:"
- board text added: "Dielectric 1"
- board text added: "Dielectric 2"
- board text added: "Dielectric 3"
- board text added: "Edge card connectors:"
- board text added: "Epsilon R"
- board text added: "F.Cu"
- board text added: "F.Mask"
- board text added: "F.Paste"
- board text added: "F.Silkscreen"
- board text added: "FR4"
- board text added: "IMPEDANCE TABLE UNIT :MM"
- board text added: "IN2"
- board text added: "Impedance Control:"
- board text added: "In1.Cu"
- board text added: "In2.Cu"
- board text added: "LAYER"
- board text added: "Layer Name"
- board text added: "Loss Tangent"
- board text added: "Material"
- board text added: "Min hole diameter:"
- board text added: "Min track/spacing:"
- board text added: "No"
- board text added: "None"
- board text added: "Not specified"
- board text added: "Plated Board Edge:"
- board text added: "Silkscreen Color : White Soldermask : Matte Black Follow IPC Class 2"
- board text added: "TOP"
- board text added: "Thickness (mm)"
- board text added: "Top Silk Screen"
- board text added: "Top Solder Mask"
- board text added: "Top Solder Paste"
- board text added: "Type"
- board text added: "WIDTH"
- board text added: "WIDTH SPACING"
- board text added: "Yes"
- board text added: "copper"
- board text added: "core"
- board text added: "prepreg"

Commit message: Changed loading caps to 10pF, changed HSTX port naming to be consistent with other RPi boards with no routing changes, added docs for FPC connector
Parts:
- LOGO4: value OSHW ID: US002140 -> OSHW ID: US002732
Changed lines of the file:
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@@
 		(grid_origin 58.455718 114.689071)
 		(pcbplotparams
-			(layerselection 0x003f0fc_ffffffff)
+			(layerselection 0x00311fc_ffffffff)
 			(plot_on_all_layers_selection 0x0001000_00000000)
 			(disableapertmacros no)
@@
 			(drillshape 0)
 			(scaleselection 1)
-			(outputdirectory "Fabrication/Gerber/")
+			(outputdirectory "Fabrication_pico2-ice/Assembly/")
 		)
 	)
@@
 			)
 		)
-		(property "Value" "OSHW ID: US002140"
+		(property "Value" "OSHW ID: US002732"
 			(at -0.3302 1.9558 0)
 			(layer "B.Mask")
@@
 		)
 		(property "Value" "10K"
-			(at -1.338129 1.204118 270)
+			(at -1.338129 1.204118 -90)
 			(layer "F.Fab")
 			(hide yes)
@@
 		)
 		(property "Footprint" "Resistor_SMD:R_0402_1005Metric"
-			(at 0 0 270)
+			(at 0 0 -90)
 			(layer "B.Fab")
 			(hide yes)
@@
 		)
 		(property "Datasheet" ""
-			(at 0 0 270)
+			(at 0 0 -90)
 			(layer "B.Fab")
 			(hide yes)
@@
 		)
 		(fp_text user "${REFERENCE}"
-			(at 0 0 270)
+			(at 0 0 -90)
 			(layer "F.Fab")
 			(effects
@@
 		)
 		(property "Value" "4.7u"
-			(at 0 -1.16 360)
+			(at 0 -1.16 0)
 			(layer "B.Fab")
 			(hide yes)
@@
 		)
 		(property "Footprint" "Capacitor_SMD:C_0402_1005Metric"
-			(at 0 0 360)
+			(at 0 0 0)
 			(layer "B.Fab")
 			(hide yes)
@@
 		)
 		(property "Datasheet" ""
-			(at 0 0 360)
+			(at 0 0 0)
 			(layer "B.Fab")
 			(hide yes)
@@
 		)
 		(fp_text user "${REFERENCE}"
-			(at 0 0 360)
+			(at 0 0 0)
 			(layer "B.Fab")
 			(effects
@@
 	)
 	(gr_line
-		(start 83.82 77.47)
-		(end 83.82 130.81)
+		(start 86.955035 74.399754)
+		(end 86.902626 131.125979)
+		(stroke
+			(width 0.127)
+			(type solid)
+		)
+		(layer "B.Fab")
+	)
+	(gr_line
+		(start 62.955041 75.29976)
+		(end 62.902632 132.025985)
+		(stroke
+			(width 0.127)
+			(type solid)
+		)
+		(layer "B.Fab")
+	)
+	(gr_line
+		(start 61.755718 70.589071)
+		(end 83.175718 70.589071)
+		(stroke
+			(width 0.127)
+			(type solid)
+		)
+		(layer "B.Fab")
+	)
+	(gr_arc
+		(start 59.145041 71.48976)
+		(mid 61.855724 72.589077)
+		(end 62.955041 75.29976)
+		(stroke
+			(width 0.127)
+			(type solid)
+		)
+		(layer "B.Fab")
+	)
+	(gr_line
+		(start 33.855724 71.789077)
+		(end 55.275724 71.789077)
+		(stroke
+			(width 0.127)
+			(type solid)
+		)
+		(layer "B.Fab")
+	)
+	(gr_arc
+		(start 33.81881 136.135985)
+		(mid 31.155724 134.989071)
+		(end 30.00881 132.325985)
+		(stroke
+			(width 0.127)
+			(type solid)
+		)
+		(layer "B.Fab")
+	)
+	(gr_arc
+		(start 37.71881 135.835985)
+		(mid 35.055724 134.689071)
+		(end 33.90881 132.025985)
+		(stroke
+			(width 0.127)
+			(type solid)
+		)
+		(layer "B.Fab")
+	)
+	(gr_arc
+		(start 86.902626 131.125979)
+		(mid 85.755712 133.789065)
+		(end 83.092626 134.935979)
+		(stroke
+			(width 0.127)
+			(type solid)
+		)
+		(layer "B.Fab")
+	)
+	(gr_line
+		(start 57.908804 131.125979)
+		(end 57.945718 74.399071)
+		(stroke
+			(width 0.127)
+			(type solid)
+		)
+		(layer "B.Fab")
+	)
+	(gr_line
+		(start 59.055041 75.59976)
+		(end 59.002632 132.325985)
 		(stroke
 			(width 0.127)
@@
 	)
 	(gr_line
-		(start 64.77 73.66)
-		(end 80.01 73.66)
+		(start 83.092626 134.935979)
+		(end 61.81881 134.935979)
 		(stroke
 			(width 0.127)
@@
 	)
 	(gr_arc
-		(start 83.82 130.81)
-		(mid 82.673092 133.473092)
-		(end 80.01 134.62)
+		(start 33.945724 75.299077)
+		(mid 35.045041 72.588394)
+		(end 37.755724 71.489077)
 		(stroke
 			(width 0.127)
@@
 	)
 	(gr_line
-		(start 60.96 130.81)
-		(end 60.96 77.47)
+		(start 59.092632 135.835985)
+		(end 37.818816 135.835985)
 		(stroke
 			(width 0.127)
@@
 	)
 	(gr_line
-		(start 80.01 134.62)
-		(end 64.77 134.62)
+		(start 37.755724 71.489077)
+		(end 59.175724 71.489077)
+		(stroke
+			(width 0.127)
+			(type solid)
+		)
+		(layer "B.Fab")
+	)
+	(gr_line
+		(start 33.90881 132.025985)
+		(end 33.945724 75.299077)
 		(stroke
 			(width 0.127)
@@
 	)
 	(gr_arc
-		(start 80.01 73.66)
-		(mid 82.720683 74.759317)
-		(end 83.82 77.47)
+		(start 30.045724 75.599077)
+		(mid 31.145041 72.888394)
+		(end 33.855724 71.789077)
+		(stroke
+			(width 0.127)
+			(type solid)
+		)
+		(layer "B.Fab")
+	)
+	(gr_arc
+		(start 59.002632 132.325985)
+		(mid 57.855718 134.989071)
+		(end 55.192632 136.135985)
+		(stroke
+			(width 0.127)
+			(type solid)
+		)
+		(layer "B.Fab")
+	)
+	(gr_arc
+		(start 62.902632 132.025985)
+		(mid 61.755718 134.689071)
+		(end 59.092632 135.835985)
+		(stroke
+			(width 0.127)
+			(type solid)
+		)
+		(layer "B.Fab")
+	)
+	(gr_arc
+		(start 83.145035 70.589754)
+		(mid 85.855718 71.689071)
+		(end 86.955035 74.399754)
+		(stroke
+			(width 0.127)
+			(type solid)
+		)
+		(layer "B.Fab")
+	)
+	(gr_arc
+		(start 61.718804 134.935979)
+		(mid 59.055718 133.789065)
+		(end 57.908804 131.125979)
+		(stroke
+			(width 0.127)
+			(type solid)
+		)
+		(layer "B.Fab")
+	)
+	(gr_line
+		(start 55.192632 136.135985)
+		(end 33.918816 136.135985)
+		(stroke
+			(width 0.127)
+			(type solid)
+		)
+		(layer "B.Fab")
+	)
+	(gr_line
+		(start 30.00881 132.325985)
+		(end 30.045724 75.599077)
 		(stroke
 			(width 0.127)
@@
 	)
 	(gr_arc
-		(start 64.77 134.62)
-		(mid 62.106908 133.473092)
-		(end 60.96 130.81)
+		(start 57.945718 74.399071)
+		(mid 59.045035 71.688388)
+		(end 61.755718 70.589071)
 		(stroke
 			(width 0.127)
@@
 	)
 	(gr_arc
-		(start 60.96 77.47)
-		(mid 62.059317 74.759317)
-		(end 64.77 73.66)
+		(start 55.245041 71.78976)
+		(mid 57.955724 72.889077)
+		(end 59.055041 75.59976)
 		(stroke
 			(width 0.127)
